File: data/kicad/fixtures/minimal.kicad_pcb (KiCad board)
At the start: 2 copper layers, 0 parts

Commit message: test: give KiCad DRC fixture a valid board outline
Other:
- board outline added: 80 x 80 mm
Changed lines of the file:
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@@
   )
   (setup (pad_to_mask_clearance 0))
+  (gr_rect
+    (start 10 10)
+    (end 90 90)
+    (stroke (width 0.05) (type default))
+    (fill none)
+    (layer "Edge.Cuts")
+  )
 )
